File: Kicad-PCB/alice-pcb.sch (KiCad schematic (older format))
At the start: 121 parts

Commit message: Testing in handwired pcb
Parts:
- removed D? (x4): D, symbol Device:D_Small
- removed MX0A?, MX0B?, MX0C?, MX0D?: MX-NoLED, symbol MX_Alps_Hybrid:MX-NoLED
- added D40, D41, D42, D43, D46, D47, D48, D4A, D4B, D4C, D51, D52: D, symbol Device:D_Small
- added MX40, MX41, MX42, MX43, MX46, MX47, MX48, MX4A, MX4B, MX4C, MX51, MX52: MX-NoLED, symbol MX_Alps_Hybrid:MX-NoLED
- gave numbers to parts that had none: 48
Connections:
- net labels removed: col15
- wire segments 148 -> 186
